File: 05-Layout/nowae031/nowae031-0/nowae031.kicad_pcb (KiCad board)
At the start: 2 copper layers, 50 x 89.2 mm, 75 parts, among them P101 COMM, P102 SUPPLY, U101 TCA9554PWR, U102 TCA9554PWR

Commit message: WiP on PCB
Parts:
- moved G*** 104.2 mm to (130.2, 122.9)
- moved G*** 88.1 mm to (116.5, 122.7)
- moved TP104 34.7 mm to (126.0, 107.7)
- moved TP103 34.6 mm to (122.9, 107.7)
- moved VAL** 1.51 mm to (107.5, 125.0) (x2)
Routing:
- net +3.3V: track 195.3 -> 252.4 mm
- net /BRANCH_SCL: track 15.6 -> 63.6 mm, vias 2 -> 4
- net /BRANCH_SDA: track 16.4 -> 62.7 mm
- net GND: track 25.0 -> 50.4 mm, vias 0 -> 3
- net /B_LINE7: track 18.0 -> 20.9 mm
- added copper zone on B.Cu, net GND
Other:
- board text added: "NOWAE031-0"
- board text added: "SCL"
- board text added: "SDA"
